File: PCB/PCBMacropad.kicad_sch (KiCad schematic)
At the start: 12 parts, among them SW1 SW_Push, SW2 SW_Push, SW3 SW_Push, SW4 SW_Push, SW5 SW_Push, SW6 SW_Push, SW7 SW_Push, SW8 SW_Push, SW9 SW_Push, U1 XIAO-RP2040-DIP

Commit message: Add files via upload
Parts:
- removed C1: 0.1uF, Capacitor_THT:C_Disc_D3.0mm_W1.6mm_P2.50mm, symbol Device:C
Changed lines of the file:
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@@
 	(paper "A4")
-	(junction
-		(at 135.89 162.56)
-		(diameter 0)
-		(color 0 0 0 0)
-	)
 	(junction
 		(at 191.77 132.08)
@@
 	)
 	(junction
-		(at 135.89 147.32)
-		(diameter 0)
-		(color 0 0 0 0)
-	)
-	(junction
 		(at 191.77 102.87)
 		(diameter 0)
@@
 	(wire
 		(pts
-			(xy 151.13 158.75) (xy 151.13 165.1)
-		)
-		(stroke
-			(width 0)
-			(type default)
-		)
-	)
-	(wire
-		(pts
 			(xy 163.83 118.11) (xy 163.83 119.38)
 		)
@@
 	(wire
 		(pts
-			(xy 135.89 142.24) (xy 135.89 147.32)
-		)
-		(stroke
-			(width 0)
-			(type default)
-		)
-	)
-	(wire
-		(pts
 			(xy 156.21 127) (xy 166.37 127)
 		)
@@
 	(wire
 		(pts
-			(xy 151.13 142.24) (xy 135.89 142.24)
-		)
-		(stroke
-			(width 0)
-			(type default)
-		)
-	)
-	(wire
-		(pts
 			(xy 166.37 147.32) (xy 181.61 147.32)
 		)
@@
 	(wire
 		(pts
-			(xy 135.89 165.1) (xy 135.89 162.56)
-		)
-		(stroke
-			(width 0)
-			(type default)
-		)
-	)
-	(wire
-		(pts
 			(xy 175.26 132.08) (xy 175.26 123.19)
 		)
@@
 	(wire
 		(pts
-			(xy 151.13 165.1) (xy 135.89 165.1)
-		)
-		(stroke
-			(width 0)
-			(type default)
-		)
-	)
-	(wire
-		(pts
 			(xy 128.27 154.94) (xy 115.57 154.94)
 		)
@@
 			(width 0)
 			(type default)
-		)
-	)
-	(wire
-		(pts
-			(xy 151.13 142.24) (xy 151.13 151.13)
-		)
-		(stroke
-			(width 0)
-			(type default)
-		)
-	)
-	(symbol
-		(lib_id "Device:C")
-		(at 151.13 154.94 0)
-		(unit 1)
-		(exclude_from_sim no)
-		(in_bom yes)
-		(on_board yes)
-		(dnp no)
-		(fields_autoplaced yes)
-		(property "Reference" "C1"
-			(at 154.94 153.6699 0)
-			(effects
-				(font
-					(size 1.27 1.27)
-				)
-				(justify left)
-			)
-		)
-		(property "Value" "0.1uF"
-			(at 154.94 156.2099 0)
-			(effects
-				(font
-					(size 1.27 1.27)
-				)
-				(justify left)
-			)
-		)
-		(property "Footprint" "Capacitor_THT:C_Disc_D3.0mm_W1.6mm_P2.50mm"
-			(at 152.0952 158.75 0)
-			(effects
-				(font
-					(size 1.27 1.27)
-				)
-				(hide yes)
-			)
-		)
-		(property "Datasheet" "~"
-			(at 151.13 154.94 0)
-			(effects
-				(font
-					(size 1.27 1.27)
-				)
-				(hide yes)
-			)
-		)
-		(property "Description" "Unpolarized capacitor"
-			(at 151.13 154.94 0)
-			(effects
-				(font
-					(size 1.27 1.27)
-				)
-				(hide yes)
-			)
-		)
-		(pin "1"
-		)
-		(pin "2"
-		)
-		(instances
-			(project ""
-				(path "/5fddeb03-6c3a-4766-b255-fc09c5ebac1d"
-					(reference "C1")
-					(unit 1)
-				)
-			)
 		)
 	)
@@
 		(dnp no)
 		(property "Reference" "D1"
-			(at 144.018 145.288 0)
+			(at 147.828 148.336 0)
 			(effects
 				(font
@@
 		)
 		(property "Value" "SK6812MINI"
-			(at 144.018 147.828 0)
+			(at 147.828 150.876 0)
 			(effects
 				(font
@@
 		)
 		(property "Value" "+5V"
-			(at 135.89 140.208 0)
-			(effects
-				(font
+			(at 135.89 143.256 0)
+			(effects
+				(font
